File: hardware/pico-hat-version/BlackGPIB_vertical_sd.kicad_pcb (KiCad board)
At the start: 2 copper layers, 7 parts, among them J1 SD_Card_Module, J2 Raspberry_Pi_Connector

Commit message: pcb
Parts:
- moved J1 8.34 mm to (213.7, 69.5), turned to -90 degrees
Routing:
- net GND: track 325.0 -> 290.9 mm
- net +3.3V: track 30.4 -> 46.7 mm
- net SPI_MOSI: track 6.16 -> 14.4 mm
- net SPI_SCK: track 6.16 -> 12.6 mm
- net SPI_MISO: track 7.44 -> 9.11 mm
- net SPI_CS: track 16.1 -> 17.5 mm
