File: hardware/pi-hat/untitled.kicad_pcb (KiCad board)
At the start: 2 copper layers, 75 x 65 mm, 61 parts, among them IC3 75161P, IC4 75161SO, IC5 75162P, IC6 75162P1, IC7 75162SO24

Commit message: pi: swap srq and atn on the gpib hat and fix import issues
Parts:
- C1, C2: value (none) -> C-EUC0805
- C3, C4: value (none) -> C-EU050-024X044
- IC1: value (none) -> 75160P
- IC2: value (none) -> 75160SO
- IC6: value 75162P1 -> 75162
- JP1, JP2: value (none) -> PINHD-1X5
- JP3: value (none) -> GPIB-PINHD-2X12
- PL1: value (none) -> C24HP
- R1, R10, R11, R12, R13, R14, R15, R16, R17, R18, R19, R2, R20, R21, R22, R23, R24, R25, R26, R27, R28, R29, R3, R30, R31, R32, R33, R34, R35, R36, R37, R38, R39, R4, R40, R5, R6, R7, R8, R9: value (none) -> 3k
Connections:
- net ATN1 renamed /ATN1
- net DAV renamed /DAV
- net DAV1 renamed /DAV1
- net DC renamed /DC
- net DIO1 renamed /DIO1
- net DIO2 renamed /DIO2
- net DIO3 renamed /DIO3
- net DIO4 renamed /DIO4
- net DIO5 renamed /DIO5
- net DIO6 renamed /DIO6
- net DIO7 renamed /DIO7
- net DIO8 renamed /DIO8
- net EOI renamed /EOI
- net EOI1 renamed /EOI1
- net IFC renamed /IFC
- net IFC1 renamed /IFC1
- net IO1 renamed /IO1
- net IO2 renamed /IO2
- net IO3 renamed /IO3
- net IO4 renamed /IO4
- net IO5 renamed /IO5
- net IO6 renamed /IO6
- net IO7 renamed /IO7
- net IO8 renamed /IO8
- net NDAC renamed /NDAC
- net NDAC1 renamed /NDAC1
- net NRFD renamed /NRFD
- net NRFD1 renamed /NRFD1
- net PE renamed /PE
- net REN renamed /REN
- net REN1 renamed /REN1
- net SC renamed /SC
- net SCL renamed /SCL
- net SDA renamed /SDA
- net SRQ1 renamed /SRQ1
- net TE renamed /TE
- IC3 pad 8: ATN -> /ATN
- IC3 pad 9: SRQ -> /SRQ
- IC4 pad 8: ATN -> /ATN
- IC4 pad 9: SRQ -> /SRQ
- IC5 pad 10: SRQ -> /SRQ
- IC5 pad 21: (no net) -> unconnected-(IC5A-NC-Pad21)
- IC5 pad 9: ATN -> /ATN
- IC6 pad 10: SRQ -> /SRQ
- IC6 pad 11: (no net) -> unconnected-(IC6A-NC-Pad11)_1
- IC6 pad 14: (no net) -> unconnected-(IC6A-NC-Pad11)_2
- IC6 pad 23: (no net) -> unconnected-(IC6A-NC-Pad11)
- IC6 pad 9: ATN -> /ATN
- IC7 pad 10: SRQ -> /SRQ
- IC7 pad 11: (no net) -> unconnected-(IC7A-NC-Pad11)_2
- IC7 pad 14: (no net) -> unconnected-(IC7A-NC-Pad11)_1
- IC7 pad 23: (no net) -> unconnected-(IC7A-NC-Pad11)
- IC7 pad 9: ATN -> /ATN
- JP3 pad 10: ATN -> /SRQ
- JP3 pad 11: SRQ -> /ATN
- PL1 pad 10: ATN -> /SRQ
- PL1 pad 11: SRQ -> /ATN
- U$2 pad 10: (no net) -> unconnected-(U$2-10-RX-Pad10)
- U$2 pad 12: (no net) -> unconnected-(U$2-12-GPIO18-Pad12)
- U$2 pad 17: (no net) -> unconnected-(U$2-17-3V3-Pad17)
- U$2 pad 27: (no net) -> unconnected-(U$2-27-ID_SD-Pad27)
- U$2 pad 28: (no net) -> unconnected-(U$2-28-ID_SC-Pad28)
- U$2 pad 7: (no net) -> unconnected-(U$2-7-GPIO4-Pad7)
- U$2 pad 8: (no net) -> unconnected-(U$2-8-TX-Pad8)
Routing:
- net ATN: track 35.2 -> 0.00 mm, vias 1 -> 0
- net SRQ: track 32.7 -> 0.00 mm
- net /SRQ: track 0.00 -> 30.3 mm
- net /ATN: track 0.00 -> 28.7 mm
- net /DC: track 24.5 -> 0.00 mm
- net (no net): track 0.00 -> 24.5 mm
