File: hardware/pi-hat/untitled.kicad_sch (KiCad schematic)
At the start: 57 parts, among them IC1 75160P, IC2 75160SO, IC3 75161P, IC4 75161SO, IC5 75162P, IC6 75162, IC7 75162SO24

Commit message: pi: swap srq and atn on the gpib hat and fix import issues
Parts:
- R1, R10, R11, R12, R13, R14, R15, R16, R17, R18, R19, R2, R20, R3, R4, R5, R6, R7, R8, R9: value R-EU_R0805 -> 3k
- R21, R22, R23, R24, R25, R26, R27, R28, R29, R30, R31, R32, R33, R34, R35, R36, R37, R38, R39, R40: value R-EU_0204/7 -> 3k
Connections:
- net ATN: now also JP3.11, PL1.11; no longer JP3.10, PL1.10
- net NDAC: no longer IC3.5 (NRFD2), IC4.5 (NRFD2), IC5.6 (NRFD2), IC6.6 (NRFD2), IC7.6 (NRFD2), JP3.7, PL1.7
- net SRQ: now also JP3.10, PL1.10; no longer JP3.11, PL1.11
- new net NRFD: IC3.5 (NRFD2), IC4.5 (NRFD2), IC5.6 (NRFD2), IC6.6 (NRFD2), IC7.6 (NRFD2), JP3.7, PL1.7
- no-connect marks 0 -> 3
