File: hardware/pico/BlackGPIB Pico.kicad_pcb (KiCad board)
At the start: 2 copper layers, 66.2 x 60.9 mm, 20 parts, among them J3 Micro_SD_Card, U1 SN75160, U2 SN75160, U3 SN75161, U4 SN75161, U5 SN75162, U6 SN75162

Commit message: pico: add 47uF tantalum capacitor near sd card slot to rev 1 board
Parts:
- added C4: 47uF, Capacitor_Tantalum_SMD:CP_EIA-6032-15_Kemet-U_HandSolder, B.Cu at (113.4, 94.6)
Routing:
- net +3.3V: track 34.3 -> 37.8 mm
Changed lines of the file:
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@@
 		)
 	)
+	(footprint "Capacitor_Tantalum_SMD:CP_EIA-6032-15_Kemet-U_HandSolder"
+		(layer "B.Cu")
+		(at 113.411 94.6325 -90)
+		(descr "Tantalum Capacitor SMD Kemet-U (6032-15 Metric), IPC-7352 nominal, (Body size from: http://www.kemet.com/Lists/ProductCatalog/Attachments/253/KEM_TC101_STD.pdf), generated with kicad-footprint-generator")
+		(tags "capacitor tantalum")
+		(property "Reference" "C4"
+			(at 0 2.55 90)
+			(layer "B.SilkS")
+			(hide yes)
+			(effects
+				(font
+					(size 1 1)
+					(thickness 0.15)
+				)
+				(justify mirror)
+			)
+		)
+		(property "Value" "47uF"
+			(at 0 -2.55 90)
+			(layer "B.SilkS")
+			(effects
+				(font
+					(size 1 1)
+					(thickness 0.15)
+				)
+				(justify mirror)
+			)
+		)
+		(property "Datasheet" "~"
+			(at 0 0 90)
+			(layer "B.Fab")
+			(hide yes)
+			(effects
+				(font
+					(size 1.27 1.27)
+					(thickness 0.15)
+				)
+				(justify mirror)
+			)
+		)
+		(property "Description" "Polarized capacitor"
+			(at 0 0 90)
+			(layer "B.Fab")
+			(hide yes)
+			(effects
+				(font
+					(size 1.27 1.27)
+					(thickness 0.15)
+				)
+				(justify mirror)
+			)
+		)
+		(property ki_fp_filters "CP_*")
+		(sheetname "/")
+		(sheetfile "BlackGPIB Pico.kicad_sch")
+		(attr smd)
+		(fp_line
+			(start -3.94 1.71)
+			(end -3.94 -1.71)
+			(stroke
+				(width 0.12)
+				(type solid)
+			)
+			(layer "B.SilkS")
+		)
+		(fp_line
+			(start 3 1.71)
+			(end -3.94 1.71)
+			(stroke
+				(width 0.12)
+				(type solid)
+			)
+			(layer "B.SilkS")
+		)
+		(fp_line
+			(start -3.94 -1.71)
+			(end 3 -1.71)
+			(stroke
+				(width 0.12)
+				(type solid)
+			)
+			(layer "B.SilkS")
+		)
+		(fp_rect
+			(start -3.93 1.85)
+			(end 3.93 -1.85)
+			(stroke
+				(width 0.05)
+				(type solid)
+			)
+			(fill no)
+			(layer "B.CrtYd")
+		)
+		(fp_line
+			(start -2.2 1.6)
+			(end -3 0.8)
+			(stroke
+				(width 0.1)
+				(type solid)
+			)
+			(layer "B.Fab")
+		)
+		(fp_line
+			(start 3 1.6)
+			(end -2.2 1.6)
+			(stroke
+				(width 0.1)
+				(type solid)
+			)
+			(layer "B.Fab")
+		)
+		(fp_line
+			(start -3 0.8)
+			(end -3 -1.6)
+			(stroke
+				(width 0.1)
+				(type solid)
+			)
+			(layer "B.Fab")
+		)
+		(fp_line
+			(start -3 -1.6)
+			(end 3 -1.6)
+			(stroke
+				(width 0.1)
+				(type solid)
+			)
+			(layer "B.Fab")
+		)
+		(fp_line
+			(start 3 -1.6)
+			(end 3 1.6)
+			(stroke
+				(width 0.1)
+				(type solid)
+			)
+			(layer "B.Fab")
+		)
+		(pad "1" smd roundrect
+			(at -2.5575 0 270)
+			(size 2.245 2.39)
+			(layers "B.Cu" "B.Mask" "B.Paste")
+			(roundrect_rratio 0.111359)
+			(net 5 "+3.3V")
+			(pintype "passive")
+		)
+		(pad "2" smd roundrect
+			(at 2.5575 0 270)
+			(size 2.245 2.39)
+			(layers "B.Cu" "B.Mask" "B.Paste")
+			(roundrect_rratio 0.111359)
+			(net 1 "GND")
+			(pintype "passive")
+		)
+		(embedded_fonts no)
+		(model "${KICAD9_3DMODEL_DIR}/Capacitor_Tantalum_SMD.3dshapes/CP_EIA-6032-15_Kemet-U.step"
+			(offset
+				(xyz 0 0 0)
+			)
+			(scale
+				(xyz 1 1 1)
+			)
+			(rotate
+				(xyz 0 0 0)
+			)
+		)
+	)
 	(footprint "Capacitor_SMD:C_1206_3216Metric_Pad1.33x1.80mm_HandSolder"
 		(layer "B.Cu")
@@
 	)
 	(segment
+		(start 110.5285 90.551)
+		(end 111.887 90.551)
+		(width 0.6)
+		(layer "B.Cu")
+		(net 5)
+	)
+	(segment
+		(start 111.202 87.802)
+		(end 111.202 88.569)
+		(width 0.6)
+		(layer "B.Cu")
+		(net 5)
+	)
+	(segment
+		(start 111.887 90.551)
+		(end 113.411 92.075)
+		(width 0.6)
+		(layer "B.Cu")
+		(net 5)
+	)
+	(segment
 		(start 110.49 91.948)
 		(end 110.49 90.5895)
@@
 	)
 	(segment
-		(start 111.202 89.8775)
+		(start 110.5285 89.2425)
 		(end 110.5285 90.551)
 		(width 0.6)
@@
 	)
 	(segment
-		(start 111.202 87.802)
-		(end 111.202 89.8775)
+		(start 111.202 88.569)
+		(end 110.5285 89.2425)
 		(width 0.6)
 		(layer "B.Cu")
@@
 		(min_thickness 0.1)
 		(filled_areas_thickness no)
-		(fill
+		(fill yes
 			(thermal_gap 0.5)
 			(thermal_bridge_width 0.5)

Commit message: pico: fix disconnected pads and zones on rev 1 board
Routing:
- net Net-(A1-GPIO7): track 2.41 -> 12.6 mm
- net Net-(A1-GPIO6): track 2.40 -> 12.0 mm
- net PI_DC: track 57.4 -> 51.6 mm
- net Net-(A1-GPIO5): track 2.41 -> 8.13 mm
- net Net-(A1-GPIO4): track 2.40 -> 6.76 mm
- net Net-(A1-GPIO3): track 5.23 -> 6.42 mm
- net Net-(A1-GPIO2): track 5.19 -> 6.38 mm
- net Net-(A1-GPIO1): track 8.68 -> 9.87 mm
- net GND: vias 0 -> 23
Other:
- board text added: "SN75160"
- board text added: "SN75161 or SN75162"
